Commit message: send jog command from Rviz

File: urdf/laser.urdf.xacro (robot description, xacro)
@@ -28,6 +28,6 @@
         <color rgba="0.50196 0.50196 0.50196 1"/>
     </material>
-    <material name="dark red">
-        <color rgba="0.6 0 0 1"/>
+    <material name="brown">
+        <color rgba="0.54902 0.27059 0.02745 1"/>
     </material>
     <material name="white">
@@ -112,5 +112,5 @@
                 <box size="${rail_width} ${y_rail_length} ${rail_width}"/>
             </geometry>
-            <material name="dark red"/>
+            <material name="brown"/>
         </visual>
     </link>
@@ -128,5 +128,5 @@
                 <box size="${rail_width} ${y_rail_length} ${rail_width}"/>
             </geometry>
-            <material name="dark red"/>
+            <material name="brown"/>
         </visual>
     </link>
@@ -142,5 +142,5 @@
                 <box size="${x_rail_length} ${rail_width} ${rail_width}"/>
             </geometry>
-            <material name="dark red"/>
+            <material name="brown"/>
         </visual>
     </link>

Commit message: add Z axis jog

File: urdf/laser.urdf.xacro (robot description, xacro)
@@ -53,9 +53,9 @@
         </visual>
     </link>
-    <joint name="base_link__rotary_base" type="fixed">
+    <joint name="rotary_base__base_link" type="fixed">
         <axis xyz="0 0 1" />
-        <origin rpy="0 0 0" xyz="0.020 0 0"/>
-        <parent link="base_link"/>
-        <child link="rotary_base"/>
+        <origin rpy="0 0 0" xyz="-0.020 0 0"/>
+        <parent link="rotary_base"/>
+        <child link="base_link"/>
     </joint>
     <link name="rotary_base_invisible">
@@ -118,7 +118,7 @@
         <axis xyz="0 0 1" />
         <limit effort="1000.0" lower="${Z_limit}" upper="0" velocity="1" />
-        <origin rpy="0 0 0" xyz="${rotary_center_to_linear_stage_x + X_joint_offset + rail_width/2} ${rotary_center_to_linear_stage_y - Y_joint_offset + rail_width/2 + laser_rad} ${metal_plate_to_rotary_center_height + rotary_center_to_linear_stage_z + laser_height - 1.5*rail_width}"/>
-        <parent link="rotary_base"/>
-        <child link="y_box1"/>
+        <origin rpy="0 0 0" xyz="${-rotary_center_to_linear_stage_x - X_joint_offset - rail_width/2} ${-rotary_center_to_linear_stage_y + Y_joint_offset - rail_width/2 - laser_rad} ${-metal_plate_to_rotary_center_height - rotary_center_to_linear_stage_z - laser_height + 1.5*rail_width}"/>
+        <parent link="y_box1"/>
+        <child link="rotary_base"/>
     </joint>
     <link name="y_box2">
@@ -152,8 +152,8 @@
         <child link="x_box"/>
     </joint>
-    <!-- tool = Tool Coordinates Frame -->
+    <!-- Tool Coordinates Frame -->
     <link name="T">
         <visual>
-            <origin rpy="0 0 0" xyz="0 0 ${laser_height/2}"/>
+            <origin rpy="0 0 0" xyz="0 0 ${-laser_height/2}"/>
             <geometry>
                 <cylinder radius="${laser_rad}" length="${laser_height}"/>
@@ -164,5 +164,5 @@
         <axis xyz="1 0 0" />
         <limit effort="1000.0" lower="${X_limit}" upper="0" velocity="1" />
-        <origin rpy="0 0 3.1415" xyz="${X_joint_offset} ${rail_width/2+laser_rad} ${rail_width/2-laser_height}"/>
+        <origin rpy="3.1415 0 3.1415" xyz="${X_joint_offset} ${rail_width/2+laser_rad} ${rail_width/2-laser_height}"/>
         <parent link="x_box"/>
         <child link="T"/>

Commit message: complete links measurement

File: urdf/laser.urdf.xacro (robot description, xacro)
@@ -2,11 +2,12 @@
 <robot name="laser" xmlns:xacro="http://www.ros.org/wiki/xacro">
     <!-- Modele Parameters (m)-->
-    <xacro:property name="metal_plate_length" value="0.43"/>
-    <xacro:property name="metal_plate_width" value="0.20"/>
-    <xacro:property name="metal_plate_to_rotary_center_height" value="0.080"/>
-    <xacro:property name="rotary_center_to_rotary_top" value="0.1263"/>
-    <xacro:property name="rotary_center_to_linear_stage_x" value="0.102"/>
-    <xacro:property name="rotary_center_to_linear_stage_y" value="-0.207"/>
-    <xacro:property name="rotary_center_to_linear_stage_z" value="0.2186"/>
+    <xacro:property name="base_plate_length" value="0.43"/>
+    <xacro:property name="base_plate_width" value="0.20"/>
+    <xacro:property name="base_plate_thickness" value="0.003"/>
+    <xacro:property name="base_plate_to_rotary_center_height" value="0.080"/>
+    <xacro:property name="rotary_center_to_rotary_top" value="0.125"/>
+    <xacro:property name="rotary_center_to_laser_head_x" value="0.103"/>
+    <xacro:property name="rotary_center_to_laser_head_y" value="0.210"/>
+    <xacro:property name="rotary_center_to_laser_head_z" value="0.214"/>
     <xacro:property name="laser_rad" value="0.015"/>
     <xacro:property name="laser_height" value="0.069"/>
@@ -15,11 +16,10 @@
     <xacro:property name="x_rail_length" value="0.347"/>
     <!-- Joint Parameters -->
-    <xacro:property name="X_limit" value="-0.290"/>
+    <xacro:property name="X_limit" value="-0.280"/>
     <xacro:property name="Y_limit" value="-0.280"/>
     <xacro:property name="Z_limit" value="-0.065"/>
     <xacro:property name="A_limit" value="-2.617"/>
-    <xacro:property name="B_limit" value="-62.8"/>
-    <xacro:property name="Y_joint_offset" value="0.08"/>
-    <xacro:property name="X_joint_offset" value="0.03"/>
+    <xacro:property name="X_joint_initial_offset" value="0.03"/>
+    <xacro:property name="Y_joint_initial_offset" value="0.08"/>
     <material name="blue">
         <color rgba="0 0 0.8 1"/>
@@ -34,14 +34,5 @@
         <color rgba="1 1 1 1"/>
     </material>
-    <link name="base_link">
-        <visual>
-            <origin rpy="0 0 0" xyz="0 0 -0.0015"/>
-            <geometry>
-                <box size="${metal_plate_length} ${metal_plate_width} 0.003"/>
-            </geometry>
-            <material name="blue"/>
-        </visual>
-    </link>
-    <!-- Rotary Table -->
+    <!-- Rotary Base Frame is at the bottom of ratary platform -->
     <link name="rotary_base">
         <visual>
@@ -53,4 +44,15 @@
         </visual>
     </link>
+    <!-- base_link is the Z-table moving up and down -->
+    <link name="base_link">
+        <visual>
+            <!-- origin is at base plate's top center -->
+            <origin rpy="0 0 0" xyz="0 0 ${-base_plate_thickness/2}"/>
+            <geometry>
+                <box size="${base_plate_length} ${base_plate_width} ${base_plate_thickness}"/>
+            </geometry>
+            <material name="blue"/>
+        </visual>
+    </link>
     <joint name="rotary_base__base_link" type="fixed">
         <axis xyz="0 0 1" />
@@ -58,17 +60,4 @@
         <parent link="rotary_base"/>
         <child link="base_link"/>
-    </joint>
-    <link name="rotary_base_invisible">
-        <visual>
-            <origin rpy="0 0 0" xyz="0 0 0"/>
-            <geometry>
-                <box size="0 0 0"/>
-            </geometry>
-        </visual>
-    </link>
-    <joint name="rotary_base__rotary_base_invisible" type="fixed">
-        <origin rpy="1.57 0 0" xyz="0 0 0"/>
-        <parent link="rotary_base"/>
-        <child link="rotary_base_invisible"/>
     </joint>
     <link name="rotary_middle">
@@ -81,12 +70,13 @@
         </visual>
     </link>
+    <!-- A axis -->
     <joint name="A" type="revolute">
         <axis xyz="1 0 0" />
         <limit effort="1000.0" lower="${A_limit}" upper="0" velocity="1" />
-        <origin rpy="0 0 0" xyz="0 ${metal_plate_to_rotary_center_height} 0"/>
-        <parent link="rotary_base_invisible"/>
+        <origin rpy="1.588 0 0" xyz="0 0 ${base_plate_to_rotary_center_height}"/>
+        <parent link="rotary_base"/>
         <child link="rotary_middle"/>
     </joint>
-    <!-- rotary_top = Work Coordinate Frame -->
+    <!-- rotary_top is the Workpiece Frame (W) -->
     <link name="W">
         <visual>
@@ -98,12 +88,13 @@
         </visual>
     </link>
+    <!-- B axis -->
     <joint name="B" type="revolute">
         <axis xyz="0 0 1" />
-        <limit effort="1000.0" lower="${B_limit}" upper="0" velocity="1" />
+        <limit effort="1000.0" lower="0" upper="0" velocity="1" />
         <origin rpy="0 0 0" xyz="0 0 ${rotary_center_to_rotary_top}"/>
         <parent link="rotary_middle"/>
         <child link="W"/>
     </joint>
-    <!-- Linear Stage -->
+    <!-- Linear Stage y_box1 is the global fixed frame -->
     <link name="y_box1">
         <visual>
@@ -115,8 +106,9 @@
         </visual>
     </link>
+    <!-- Z axis -->
     <joint name="Z" type="prismatic">
         <axis xyz="0 0 1" />
         <limit effort="1000.0" lower="${Z_limit}" upper="0" velocity="1" />
-        <origin rpy="0 0 0" xyz="${-rotary_center_to_linear_stage_x - X_joint_offset - rail_width/2} ${-rotary_center_to_linear_stage_y + Y_joint_offset - rail_width/2 - laser_rad} ${-metal_plate_to_rotary_center_height - rotary_center_to_linear_stage_z - laser_height + 1.5*rail_width}"/>
+        <origin rpy="0 0 0" xyz="${-rotary_center_to_laser_head_x - X_joint_initial_offset - rail_width/2} ${rotary_center_to_laser_head_y + Y_joint_initial_offset - rail_width/2 - laser_rad} ${-base_plate_to_rotary_center_height - rotary_center_to_laser_head_z - laser_height + 1.5*rail_width}"/>
         <parent link="y_box1"/>
         <child link="rotary_base"/>
@@ -138,5 +130,5 @@
     <link name="x_box">
         <visual>
-            <origin rpy="0 0 0" xyz="${x_rail_length/2} 0 0"/>
+            <origin rpy="0 0 0" xyz="${-x_rail_length/2} 0 0"/>
             <geometry>
                 <box size="${x_rail_length} ${rail_width} ${rail_width}"/>
@@ -145,8 +137,9 @@
         </visual>
     </link>
+    <!-- Y axis -->
     <joint name="Y" type="prismatic">
         <axis xyz="0 1 0" />
         <limit effort="1000.0" lower="${Y_limit}" upper="0" velocity="1" />
-        <origin rpy="0 0 3.1415" xyz="${-rail_width/2} ${Y_joint_offset} ${rail_width}"/>
+        <origin rpy="0 0 0" xyz="${-rail_width/2} ${Y_joint_initial_offset} ${rail_width}"/>
         <parent link="y_box1"/>
         <child link="x_box"/>
@@ -161,8 +154,9 @@
         </visual>
     </link>
+    <!-- X axis -->
     <joint name="X" type="prismatic">
         <axis xyz="1 0 0" />
         <limit effort="1000.0" lower="${X_limit}" upper="0" velocity="1" />
-        <origin rpy="3.1415 0 3.1415" xyz="${X_joint_offset} ${rail_width/2+laser_rad} ${rail_width/2-laser_height}"/>
+        <origin rpy="3.1415 0 0" xyz="${-X_joint_initial_offset} ${-rail_width/2-laser_rad} ${rail_width/2-laser_height}"/>
         <parent link="x_box"/>
         <child link="T"/>

Commit message: created a grbl_gui launch file

File: urdf/laser.urdf.xacro (robot description, xacro)
@@ -15,4 +15,7 @@
     <xacro:property name="y_rail_length" value="0.42"/>
     <xacro:property name="x_rail_length" value="0.347"/>
+    <xacro:property name="sensor_offset_from_T_x" value="0.02"/>
+    <xacro:property name="sensor_offset_from_T_y" value="0.0"/>
+    <xacro:property name="sensor_offset_from_T_z" value="0.0"/>
     <!-- Joint Parameters -->
     <xacro:property name="X_limit" value="-0.280"/>
@@ -162,3 +165,18 @@
         <child link="T"/>
     </joint>
+    <!-- Distance Sensor Frame -->
+    <link name="sensor">
+        <visual>
+            <origin rpy="0 0 0" xyz="0 0 ${-0.005}"/>
+            <geometry>
+                <cylinder radius="${0.0025}" length="${0.01}"/>
+            </geometry>
+        </visual>
+    </link>
+    <joint name="T__sensor" type="fixed">
+        <axis xyz="1 0 0" />
+        <origin rpy="0 -1.57 0" xyz="${sensor_offset_from_T_x} ${sensor_offset_from_T_y} ${sensor_offset_from_T_z}"/>
+        <parent link="T"/>
+        <child link="sensor"/>
+    </joint>
 </robot>

Commit message: add ODmini distance sensor STL model for visulization in Rviz

File: urdf/laser.urdf.xacro (robot description, xacro)
@@ -15,7 +15,7 @@
     <xacro:property name="y_rail_length" value="0.42"/>
     <xacro:property name="x_rail_length" value="0.347"/>
-    <xacro:property name="sensor_offset_from_T_x" value="0.02"/>
+    <xacro:property name="sensor_offset_from_T_x" value="0.027"/>
     <xacro:property name="sensor_offset_from_T_y" value="0.0"/>
-    <xacro:property name="sensor_offset_from_T_z" value="0.0"/>
+    <xacro:property name="sensor_offset_from_T_z" value="0.014"/>
     <!-- Joint Parameters -->
     <xacro:property name="X_limit" value="-0.280"/>
@@ -36,4 +36,7 @@
     <material name="white">
         <color rgba="1 1 1 1"/>
+    </material>
+    <material name="black">
+        <color rgba="0.2 0.2 0.2 1"/>
     </material>
     <!-- Rotary Base Frame is at the bottom of ratary platform -->
@@ -168,8 +171,9 @@
     <link name="sensor">
         <visual>
-            <origin rpy="0 0 0" xyz="0 0 ${-0.005}"/>
+            <origin rpy="0 0 0" xyz="0 0 0"/>
             <geometry>
-                <cylinder radius="${0.0025}" length="${0.01}"/>
+                <mesh filename="package://grbl_ros2_gui/meshes/ODminiDistanceSensor.STL"/>
             </geometry>
+            <material name="black"/>
         </visual>
     </link>
